File: SMA-Q2 replacement board.sch (EAGLE design)
At the start: 69 parts, among them IC2 GD25Q16, M1 TPSTP09R, M2 TPSTP09R, Q1 MOSFET-NCHANNEL2N7002PW, U1 MOSFET-PCHANNEL_DUAL563, U2 AP2112(3.3V), U3 MCP73831T-2ACI/OT, U4 MOSFET-PCHANNEL_DUAL563, Y2 32.768

Commit message: Add files via upload
Parts:
- removed A2: TPSTP09R, testpad:TPSTP09R
Connections:
- removed net A2: A2.PP, MDBT1.P0.30/AIN6
- net CH_STAT: now also MDBT1.P0.30/AIN6
Changed lines of the file:
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@@
 <part name="U$45" library="HR_pads" deviceset="HR_PADS" device=""/>
 <part name="RST" library="testpad" deviceset="TPS" device="TP09R"/>
-<part name="A2" library="testpad" deviceset="TPS" device="TP09R"/>
 <part name="U$46" library="microbuilder" deviceset="GND" device=""/>
 <part name="SJ3" library="SparkFun-Retired" deviceset="SOLDERJUMPER" device="NO"/>
@@
 <instance part="U$45" gate="G$1" x="129.54" y="-50.8"/>
 <instance part="RST" gate="G$1" x="218.44" y="88.9" rot="R270"/>
-<instance part="A2" gate="G$1" x="121.92" y="86.36" rot="R90"/>
 <instance part="U$46" gate="G$1" x="38.1" y="-40.64">
 <attribute name="VALUE" x="36.576" y="-43.18" size="1.27" layer="96"/>
@@
 </segment>
 </net>
-<net name="A2" class="0">
-<segment>
-<pinref part="MDBT1" gate="G$1" pin="P0.30/AIN6"/>
-<wire x1="137.16" y1="86.36" x2="124.46" y2="86.36" width="0.1524" layer="91"/>
-<label x="134.62" y="86.36" size="1.778" layer="95" rot="R180"/>
-<pinref part="A2" gate="G$1" pin="PP"/>
-</segment>
-</net>
 <net name="VDIV" class="0">
 <segment>
@@
 <label x="45.72" y="187.96" size="1.778" layer="95"/>
 </segment>
-</net>
+<segment>
+<pinref part="MDBT1" gate="G$1" pin="P0.30/AIN6"/>
+<wire x1="137.16" y1="86.36" x2="124.46" y2="86.36" width="0.1524" layer="91"/>
+<label x="134.62" y="86.36" size="1.778" layer="95" rot="R180"/>
+</segment>
+</net>
